Commit message: homework 3 and 4

File: arm_description/urdf/arm.transmission.xacro (robot description, xacro)
@@ -1,7 +1,6 @@
 <?xml version="1.0"?>
 <robot xmlns:xacro="http://www.ros.org/wiki/xacro">
-  <!-- Define PositionJointInterface -->
-<xacro:macro name="arm_transmission" params="hardware_interface robot_name">
-   <transmission name="${robot_name}_tran_0">
+  <xacro:macro name="arm_transmission" params="hardware_interface robot_name">
+    <transmission name="${robot_name}_tran_0">
       <robotNamespace>/${robot_name}</robotNamespace>
       <type>transmission_interface/SimpleTransmission</type>
@@ -14,5 +13,5 @@
       </actuator>
     </transmission>
-     <transmission name="${robot_name}_tran_1">
+    <transmission name="${robot_name}_tran_1">
       <robotNamespace>/${robot_name}</robotNamespace>
       <type>transmission_interface/SimpleTransmission</type>
@@ -25,5 +24,5 @@
       </actuator>
     </transmission>
-     <transmission name="${robot_name}_tran_2">
+    <transmission name="${robot_name}_tran_2">
       <robotNamespace>/${robot_name}</robotNamespace>
       <type>transmission_interface/SimpleTransmission</type>
@@ -36,5 +35,5 @@
       </actuator>
     </transmission>
-     <transmission name="${robot_name}_tran_3">
+    <transmission name="${robot_name}_tran_3">
       <robotNamespace>/${robot_name}</robotNamespace>
       <type>transmission_interface/SimpleTransmission</type>
@@ -47,4 +46,4 @@
       </actuator>
     </transmission>
-</xacro:macro>
+  </xacro:macro>
 </robot>

File: arm_description/urdf/arm.urdf.xacro (robot description, xacro)
@@ -1,6 +1,6 @@
 <?xml version="1.0"?>
-<robot name="arm" xmlns:xacro="http://ros.org/wiki/xacro">
-<xacro:include filename="$(find arm_description)/arm.gazebo.xacro"/>
-<xacro:include filename="$(find arm_description)/urdf/arm.transmission.xacro"/>
+<robot name="arm" xmlns:xacro="http://www.ros.org/wiki/xacro">
+<xacro:include filename="$(find arm_description)/urdf/arm.gazebo.xacro" />
+<xacro:include filename="$(find arm_description)/urdf/arm.transmission.xacro" />
 <xacro:arg name="hardware_interface" default="PositionJointInterface"/>
 <xacro:arg name="robot_name" default="arm"/>
@@ -32,21 +32,21 @@
   <origin xyz="0.1 0 0" rpy="0 0 0" />
 </joint>
-<link name="base_link">
-    <visual>
-	<geometry>
-	    <box size="0.1 0.1 0.1"/>
-	</geometry>
-	<origin rpy="0 0 0" xyz="0 0 0"/>
-    </visual>
-    <collision>
-	<geometry>
-	    <box size="0.1 0.1 0.1"/>
-	</geometry>
-	<origin rpy="0 0 0" xyz="0 0 0"/>
-    </collision>
-    <inertial>
-	<mass value="0.1"/>
-	<inertia ixx="1.06682889e+08" ixy="0.0" ixz="0.0" iyy="9.92165844e+07" iyz="0.0" izz="1.26939175e+08"/>
-    </inertial>
+  <link name="base_link">
+  <visual>
+    <geometry>
+      <mesh filename="package://arm_description/meshes/base_link.stl" scale="0.001 0.001 0.001"/>
+    </geometry>
+    <origin rpy="0 0 0" xyz="0 0 0"/>
+  </visual>
+  <collision>
+    <geometry>
+      <box size="0.1 0.1 0.1"/> <!-- Replace with your desired size -->
+    </geometry>
+    <origin rpy="0 0 0" xyz="0 0 0"/>
+  </collision>
+  <inertial>
+    <mass value="0.1"/>
+    <inertia ixx="1.06682889e+08" ixy="0.0" ixz="0.0" iyy="9.92165844e+07" iyz="0.0" izz="1.26939175e+08"/>
+  </inertial>
 </link>
   <joint name="base_1_2" type="fixed">
@@ -55,5 +55,5 @@
     <origin xyz="-0.0011 -0.011 0.05"/>
   </joint>
-<link name="base_turn">
+  <link name="base_turn">
     <visual>
       <geometry>
@@ -381,5 +381,5 @@
     </inertial>
   </link>
-<xacro:arm_gazebo/>
+<xacro:arm_gazebo_tags />
 <xacro:arm_transmission hardware_interface="$(arg hardware_interface)" robot_name="$(arg robot_name)"/>
 </robot>

File: rl_fra2mo_description/urdf/fra2mo.xacro (robot description, xacro)
@@ -3,5 +3,5 @@
   <xacro:include filename="$(find rl_fra2mo_description)/urdf/fra2mo_base_macro.xacro" />
   <xacro:include filename="$(find rl_fra2mo_description)/urdf/lidar_gazebo_macro.xacro" />
-  <!-- <xacro:include filename="$(find rl_fra2mo_description)/urdf/d435_gazebo_macro.xacro" />  -->
+  <xacro:include filename="$(find rl_fra2mo_description)/urdf/d435_gazebo_macro.xacro" />
   <xacro:property name="LIDAR" value="True"/>
   <xacro:property name="DEPTH" value="True"/>
@@ -14,6 +14,6 @@
   <!-- Uncomment if you want to add also a D435 camera -->
   <!-- RGBD Sensor -->
-  <!-- <xacro:if value="${DEPTH}" >
+  <xacro:if value="${DEPTH}" >
     <xacro:d435_gazebo_sensor parent="d435_link" />
-  </xacro:if>    -->
+  </xacro:if>
 </robot>
